Commit message: cap gripper cam at pad-touch (fixes R finger branch flip)

File: ur10sim/assets/pincopen/pincopen.urdf (robot description, URDF)
Before this commit: robot pincopen_try3, 10 links, 9 joints
Joints:
- joint cam_joint: limit lower=-1.44862 upper=0.97738 effort=3 velocity=10 -> lower=-1.24791 upper=0.97738 effort=3 velocity=10
